Commit message: reduce some sensors and sensor frequency

File: models/simply_diff_drive_robot/simply_diff_drive_robot.urdf (robot description, URDF)
Before this commit: robot diff_bot, 11 links, 10 joints
Links:
- removed link back_camera
- removed link imu
- removed link lidar
Joints:
- removed joint 3d_laser_scanner_joint
- removed joint back_camera_joint
- removed joint imu_joint
